Commit message: sync

File: xtd2_launch/urdf/x500_depth.urdf (robot description, URDF)
Before this commit: robot x500_depth, 7 links, 6 joints
Links:
- removed link propeller_1
- removed link propeller_2
- removed link propeller_3
- removed link propeller_4
- added link arm_front_left, mass 0.1; visual cylinder length=0.3 radius=0.01
- added link arm_front_right, mass 0.1; visual cylinder length=0.3 radius=0.01
- added link arm_rear_left, mass 0.1; visual cylinder length=0.3 radius=0.01
- added link arm_rear_right, mass 0.1; visual cylinder length=0.3 radius=0.01
- added link motor_front_left, mass 0.05; visual cylinder length=0.02 radius=0.02
- added link motor_front_right, mass 0.05; visual cylinder length=0.02 radius=0.02
- added link motor_rear_left, mass 0.05; visual cylinder length=0.02 radius=0.02
- added link motor_rear_right, mass 0.05; visual cylinder length=0.02 radius=0.02
- added link oakd_lite_base, mass 0.061; visual box size=0.0175 0.091 0.028
- added link propeller_front_left, mass 0.05; visual cylinder length=0.01 radius=0.1
- added link propeller_front_right, mass 0.05; visual cylinder length=0.01 radius=0.1
- added link propeller_rear_left, mass 0.05; visual cylinder length=0.01 radius=0.1
- added link propeller_rear_right, mass 0.05; visual cylinder length=0.01 radius=0.1
- link IMX214: mass 0.05 -> 0.01; geometry visual cylinder length=0.005 radius=0.01
- link StereoOV7251: mass 0.1 -> 0.01; geometry visual box size=0.02 0.02 0.005
Joints:
- removed joint imx214_camera_joint
- removed joint propeller_1_joint
- removed joint propeller_2_joint
- removed joint propeller_3_joint
- removed joint propeller_4_joint
- removed joint stereo_camera_joint
- added joint arm_front_left_joint: type fixed, parent base_link, child arm_front_left, origin xyz=-0.15 0.15 0.05 rpy=0 0 2.356
- added joint arm_front_right_joint: type fixed, parent base_link, child arm_front_right, origin xyz=0.15 0.15 0.05 rpy=0 0 0.785
- added joint arm_rear_left_joint: type fixed, parent base_link, child arm_rear_left, origin xyz=-0.15 -0.15 0.05 rpy=0 0 -2.356
- added joint arm_rear_right_joint: type fixed, parent base_link, child arm_rear_right, origin xyz=0.15 -0.15 0.05 rpy=0 0 -0.785
- added joint imx214_joint: type fixed, parent oakd_lite_base, child IMX214, origin xyz=0.01233 -0.03 0.01878 rpy=0 0 0
- added joint motor_front_left_joint: type fixed, parent arm_front_left, child motor_front_left, origin xyz=0 0.15 0 rpy=0 0 0
- added joint motor_front_right_joint: type fixed, parent arm_front_right, child motor_front_right, origin xyz=0 0.15 0 rpy=0 0 0
- added joint motor_rear_left_joint: type fixed, parent arm_rear_left, child motor_rear_left, origin xyz=0 0.15 0 rpy=0 0 0
- added joint motor_rear_right_joint: type fixed, parent arm_rear_right, child motor_rear_right, origin xyz=0 0.15 0 rpy=0 0 0
- added joint oakd_lite_joint: type fixed, parent base_link, child oakd_lite_base, origin xyz=0.12 0.03 0.242 rpy=0 0 0
- added joint propeller_front_left_joint: type fixed, parent motor_front_left, child propeller_front_left, origin xyz=0 0 0.01 rpy=0 0 0
- added joint propeller_front_right_joint: type fixed, parent motor_front_right, child propeller_front_right, origin xyz=0 0 0.01 rpy=0 0 0
- added joint propeller_rear_left_joint: type fixed, parent motor_rear_left, child propeller_rear_left, origin xyz=0 0 0.01 rpy=0 0 0
- added joint propeller_rear_right_joint: type fixed, parent motor_rear_right, child propeller_rear_right, origin xyz=0 0 0.01 rpy=0 0 0
- added joint stereo_ov7251_joint: type fixed, parent oakd_lite_base, child StereoOV7251, origin xyz=0.01233 -0.03 0.01878 rpy=0 0 0

Commit message: 修正点云显示

File: xtd2_launch/urdf/x500_depth.urdf (robot description, URDF)
Before this commit: robot x500_depth, 16 links, 15 joints
Links:
- removed link IMX214
- removed link StereoOV7251
- removed link oakd_lite_base
- added link OakD-Lite/base_link, mass 0.061; visual box size=0.0175 0.091 0.028
- added link OakD-Lite/base_link/IMX214, mass 0.01; visual cylinder length=0.005 radius=0.01
- added link OakD-Lite/base_link/StereoOV7251, mass 0.01; visual box size=0.02 0.02 0.005
Joints:
- joint imx214_joint: child IMX214 -> OakD-Lite/base_link/IMX214; parent oakd_lite_base -> OakD-Lite/base_link
- joint oakd_lite_joint: child oakd_lite_base -> OakD-Lite/base_link
- joint stereo_ov7251_joint: child StereoOV7251 -> OakD-Lite/base_link/StereoOV7251; parent oakd_lite_base -> OakD-Lite/base_link

Commit message: 修正tf关系

File: xtd2_launch/urdf/x500_depth.urdf (robot description, URDF)
Before this commit: robot x500_depth, 16 links, 15 joints
Links:
- removed link OakD-Lite/base_link/IMX214
- removed link OakD-Lite/base_link/StereoOV7251
- added link IMX214, mass 0.01; visual cylinder length=0.005 radius=0.01
- added link StereoOV7251, mass 0.01; visual box size=0.02 0.02 0.005
Joints:
- joint imx214_joint: child OakD-Lite/base_link/IMX214 -> IMX214
- joint stereo_ov7251_joint: child OakD-Lite/base_link/StereoOV7251 -> StereoOV7251

Commit message: 修正tf关系

File: xtd2_launch/urdf/x500_depth.urdf (robot description, URDF)
Before this commit: robot x500_depth, 16 links, 15 joints
Links:
- removed link IMX214
- removed link OakD-Lite/base_link
- removed link StereoOV7251
- removed link arm_front_left
- removed link arm_front_right
- removed link arm_rear_left
- removed link arm_rear_right
- removed link base_link
- removed link motor_front_left
- removed link motor_front_right
- removed link motor_rear_left
- removed link motor_rear_right
- removed link propeller_front_left
- removed link propeller_front_right
- removed link propeller_rear_left
- removed link propeller_rear_right
- added link x500_depth_0/IMX214, mass 0.01; visual cylinder length=0.005 radius=0.01
- added link x500_depth_0/OakD-Lite/base_link, mass 0.061; visual box size=0.0175 0.091 0.028
- added link x500_depth_0/StereoOV7251, mass 0.01; visual box size=0.02 0.02 0.005
- added link x500_depth_0/arm_front_left, mass 0.1; visual cylinder length=0.3 radius=0.01
- added link x500_depth_0/arm_front_right, mass 0.1; visual cylinder length=0.3 radius=0.01
- added link x500_depth_0/arm_rear_left, mass 0.1; visual cylinder length=0.3 radius=0.01
- added link x500_depth_0/arm_rear_right, mass 0.1; visual cylinder length=0.3 radius=0.01
- added link x500_depth_0/base_link, mass 1.5; collision box size=0.4 0.4 0.1; visual box size=0.4 0.4 0.1
- added link x500_depth_0/motor_front_left, mass 0.05; visual cylinder length=0.02 radius=0.02
- added link x500_depth_0/motor_front_right, mass 0.05; visual cylinder length=0.02 radius=0.02
- added link x500_depth_0/motor_rear_left, mass 0.05; visual cylinder length=0.02 radius=0.02
- added link x500_depth_0/motor_rear_right, mass 0.05; visual cylinder length=0.02 radius=0.02
- added link x500_depth_0/propeller_front_left, mass 0.05; visual cylinder length=0.01 radius=0.1
- added link x500_depth_0/propeller_front_right, mass 0.05; visual cylinder length=0.01 radius=0.1
- added link x500_depth_0/propeller_rear_left, mass 0.05; visual cylinder length=0.01 radius=0.1
- added link x500_depth_0/propeller_rear_right, mass 0.05; visual cylinder length=0.01 radius=0.1
Joints:
- joint arm_front_left_joint: child arm_front_left -> x500_depth_0/arm_front_left; parent base_link -> x500_depth_0/base_link
- joint arm_front_right_joint: child arm_front_right -> x500_depth_0/arm_front_right; parent base_link -> x500_depth_0/base_link
- joint arm_rear_left_joint: child arm_rear_left -> x500_depth_0/arm_rear_left; parent base_link -> x500_depth_0/base_link
- joint arm_rear_right_joint: child arm_rear_right -> x500_depth_0/arm_rear_right; parent base_link -> x500_depth_0/base_link
- joint imx214_joint: child IMX214 -> x500_depth_0/IMX214; parent OakD-Lite/base_link -> x500_depth_0/OakD-Lite/base_link
- joint motor_front_left_joint: child motor_front_left -> x500_depth_0/motor_front_left; parent arm_front_left -> x500_depth_0/arm_front_left
- joint motor_front_right_joint: child motor_front_right -> x500_depth_0/motor_front_right; parent arm_front_right -> x500_depth_0/arm_front_right
- joint motor_rear_left_joint: child motor_rear_left -> x500_depth_0/motor_rear_left; parent arm_rear_left -> x500_depth_0/arm_rear_left
- joint motor_rear_right_joint: child motor_rear_right -> x500_depth_0/motor_rear_right; parent arm_rear_right -> x500_depth_0/arm_rear_right
- joint oakd_lite_joint: child OakD-Lite/base_link -> x500_depth_0/OakD-Lite/base_link; parent base_link -> x500_depth_0/base_link
- joint propeller_front_left_joint: child propeller_front_left -> x500_depth_0/propeller_front_left; parent motor_front_left -> x500_depth_0/motor_front_left
- joint propeller_front_right_joint: child propeller_front_right -> x500_depth_0/propeller_front_right; parent motor_front_right -> x500_depth_0/motor_front_right
- joint propeller_rear_left_joint: child propeller_rear_left -> x500_depth_0/propeller_rear_left; parent motor_rear_left -> x500_depth_0/motor_rear_left
- joint propeller_rear_right_joint: child propeller_rear_right -> x500_depth_0/propeller_rear_right; parent motor_rear_right -> x500_depth_0/motor_rear_right
- joint stereo_ov7251_joint: child StereoOV7251 -> x500_depth_0/StereoOV7251; parent OakD-Lite/base_link -> x500_depth_0/OakD-Lite/base_link

Commit message: 把深度相机当雷达用

File: xtd2_launch/urdf/x500_depth.urdf (robot description, URDF)
Before this commit: robot x500_depth, 16 links, 15 joints
Joints:
- joint oakd_lite_joint: origin xyz=0.12 0.03 0.242 rpy=0 0 0 -> xyz=0.12 0.03 0.242 rpy=0 -1.57 0

Commit message: sync

File: xtd2_launch/urdf/x500_depth.urdf (robot description, URDF)
Before this commit: robot x500_depth, 16 links, 15 joints
Joints:
- joint oakd_lite_joint: origin xyz=0.12 0.03 0.242 rpy=0 -1.57 0 -> xyz=0.12 0.03 0.242 rpy=0 0 0
